Commit message: add exprienments v1

File: environments/isaac_simulation/assets/laptop/laptop.urdf (robot description, URDF)
Before this commit: robot labtop.urdf, 1 links, 0 joints
Links:
- link baseLink: mass 0.0 -> 0.1

File: environments/isaac_simulation/assets/yellow_cup/model.urdf (robot description, URDF)
Before this commit: robot model.urdf, 1 links, 0 joints
Links:
- link baseLink: mass 0.1 -> 0.0; geometry collision mesh filename=collision.obj scale=0.7 0.7 0.7; visual mesh filename=textured.obj scale=0.7 0.7 0.7
