Commit message: add objects; 10 task example ; list todos for the complete

File: environments/isaac_simulation/assets/book_3/model.urdf (robot description, URDF)
Before this commit: robot model.urdf, 1 links, 0 joints
Links:
- link baseLink: geometry collision mesh filename=collision.obj scale=1 1 1; visual mesh filename=textured.obj scale=1 1 1

File: environments/isaac_simulation/assets/bowl/model.urdf (robot description, URDF)
Before this commit: robot model.urdf, 1 links, 0 joints
Links:
- link baseLink: mass 0.0 -> 0.1

File: environments/isaac_simulation/assets/rubick/cube.urdf (robot description, URDF)
Before this commit: robot cube.urdf, 1 links, 0 joints
Links:
- link baseLink: mass 0.0 -> 0.1

File: environments/isaac_simulation/assets/yellow_cup/model.urdf (robot description, URDF)
Before this commit: robot model.urdf, 1 links, 0 joints
Links:
- link baseLink: mass 0.0 -> 0.1; geometry collision mesh filename=collision.obj scale=1 1 1; visual mesh filename=textured.obj scale=1 1 1
